File: MPXDecorder-V4_SMD/MPXDecorder-V4_SMD.kicad_sch (KiCad schematic)
At the start: 119 parts, among them J1 MPX-IN, J2 OUT-L, J3 GND, J4 OUT-R, J5 GND, J6 5V, J7 GND, Q3 2N3904, Q4 2N3904, Q5 2N3904, Q6 2N3904, U1 TC4066BFELNF, U2 NJM2747V, U3 74HC4046APW, U4 LM393, U5 74HC74D, U6 NJM2747V, U7 NJM2747V, U8 TC4066BFELNF, U9 74HC74D

Commit message: 基板設計完了
Parts:
- removed unit 2 of U1
- added unit 4 of U8
- renumbered U8 to U1, U1 to U8
Connections:
- net +5V: now also R28.1, U9.1 (~{R}), U9.10 (~{S}), U9.13 (~{R}), U9.2 (D), U9.3 (C), U9.4 (~{S}); no longer U9.1 (~{R}), U9.10 (~{S}), U9.11 (C), U9.12 (D), U9.13 (~{R}), U9.4 (~{S})
- net 38KHz-PLL-INV: now also U9.11 (C); no longer U9.3 (C)
- net GND: now also U8.10, U8.11, U8.12; no longer D2.1 (K)
- net In-phase: now also U9.12 (D); no longer U9.2 (D)
- net MONO: now also D2.1 (K), U8.13, U8.5; no longer U8.12, U8.6
- net PD: now also U2.7; no longer U2.1
- net Quadrature-phase: now also U8.6, U9.9 (Q); no longer U8.13, U9.5 (Q)
- net VCTL: now also U2.1; no longer U2.7
- net VREF_2.5V: now also U2.3 (+), U8.9; no longer U2.5 (+), U8.2
- net at R61.2, R62.1: now also U2.6 (-); no longer U2.2 (-)
- net at C41.1, R63.2, R64.1: now also U2.2 (-), U8.1, U8.3; no longer U2.6 (-), U8.10, U8.8
- net at R85.2: now also U8.4; no longer U8.11
- net at R84.2: now also U8.2; no longer U8.9
- new net: R60.2, U2.5 (+), U8.8
