File: MPXDecorder-V4_SMD/MPXDecorder-V4_SMD.kicad_pcb (KiCad board)
At the start: 4 copper layers, 73.5 x 73.6 mm, 119 parts, among them J1 MPX-IN, J2 OUT-L, J3 GND, J4 OUT-R, J5 GND, J6 5V, J7 GND, Q3 2N3904, Q4 2N3904, Q5 2N3904, Q6 2N3904, U1 TC4066BFELNF, U2 NJM2747V, U3 74HC4046APW, U4 LM393, U5 74HC74D, U6 NJM2747V, U7 NJM2747V, U8 TC4066BFELNF, U9 74HC74D

Commit message: 基板設計完了
Parts:
- C13, C17, C18, C7, R2: moved to F.Cu
- C38, C4, C50, R1, R70, R72, R81, R82, R85, RV1, TP3, TP5, U3, U5, U8, U9: moved to B.Cu
- moved C41 91.9 mm to (57.5, 105.0), turned to 90 degrees
- moved U9 91.8 mm to (57.3, 116.0)
- moved TP10 89.7 mm to (58.1, 112.6)
- moved TP9 86.1 mm to (52.9, 109.8)
- moved C50 79.5 mm to (73.0, 108.6), turned to -90 degrees
- moved U8 78.4 mm to (61.3, 105.0), turned to 90 degrees
- moved TP6 78.3 mm to (65.0, 110.7)
- moved R64 75.6 mm to (58.4, 107.7), turned to 180 degrees
- moved TP12 74.3 mm to (70.6, 110.6)
- moved R85 73.5 mm to (61.8, 110.6), turned to 180 degrees
- moved TP11 73.0 mm to (69.8, 95.0)
- moved C40 72.6 mm to (55.6, 105.9), turned to 90 degrees
- moved R80 70.1 mm to (68.0, 106.1), turned to -90 degrees
- moved R84 68.6 mm to (66.4, 106.1), turned to -90 degrees
- moved R81 67.8 mm to (69.4, 106.1), turned to -90 degrees
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Connections:
- C41 pad 1: Net-(U2B--) -> Net-(U2A--)
- D2 pad 1: GND -> /MONO
- R28 pad 1: Net-(R28-Pad1) -> +5V
- R60 pad 2: Net-(U2A-+) -> Net-(U2B-+)
- R61 pad 2: Net-(U2A--) -> Net-(U2B--)
- R62 pad 1: Net-(U2A--) -> Net-(U2B--)
- R63 pad 2: Net-(U2B--) -> Net-(U2A--)
- R64 pad 1: Net-(U2B--) -> Net-(U2A--)
- U1 pad 3: Net-(R28-Pad1) -> Net-(R66-Pad1)
- U1 pad 4: +5V -> /COMP
- U1 pad 5: /STEREO -> /In-phase
- U1 pad 6: /MONO -> /In-phase_INV
- U1 pad 8: Net-(U2B--) -> /COMP
- U1 pad 9: Net-(R84-Pad2) -> Net-(R67-Pad1)
- U2 pad 1: /PD -> /VCTL
- U2 pad 3: Net-(U2A-+) -> /VREF_2.5V
- U2 pad 5: /VREF_2.5V -> Net-(U2B-+)
- U2 pad 7: /VCTL -> /PD
- U8 pad 1: Net-(U2A-+) -> Net-(U2A--)
- U8 pad 10: Net-(U2B--) -> GND
- U8 pad 11: Net-(R85-Pad2) -> GND
- U8 pad 12: /MONO -> GND
- U8 pad 13: /Quadrature-phase -> /MONO
- U8 pad 2: /VREF_2.5V -> Net-(R84-Pad2)
- U8 pad 3: Net-(R66-Pad1) -> Net-(U2A--)
- U8 pad 4: /COMP -> Net-(R85-Pad2)
- U8 pad 5: /In-phase -> /MONO
- U8 pad 6: /In-phase_INV -> /Quadrature-phase
- U8 pad 8: /COMP -> Net-(U2B-+)
- U8 pad 9: Net-(R67-Pad1) -> /VREF_2.5V
- U9 pad 11: +5V -> /38KHz-PLL-INV
- U9 pad 12: +5V -> /In-phase
- U9 pad 2: /In-phase -> +5V
- U9 pad 3: /38KHz-PLL-INV -> +5V
- U9 pad 5: /Quadrature-phase -> unconnected-(U9A-Q-Pad5)
- U9 pad 9: unconnected-(U9B-Q-Pad9) -> /Quadrature-phase
Routing:
- net /COMP: track 0.00 -> 43.6 mm
- net /In-phase: track 0.00 -> 37.8 mm, vias 0 -> 3
- net /38KHz-PLL-INV: track 11.4 -> 46.1 mm, vias 0 -> 2
- net /38KHz-PLL: track 19.4 -> 53.0 mm, vias 4 -> 2
- net /In-phase_INV: track 6.56 -> 35.9 mm, vias 0 -> 3
- net /MONO: track 0.00 -> 28.9 mm, vias 0 -> 2
- net Net-(U4A--): track 0.00 -> 26.7 mm, vias 0 -> 4
- net /PD: track 0.00 -> 24.1 mm, vias 0 -> 2
- net /VCO-IN: track 0.00 -> 24.0 mm, vias 0 -> 1
- net /VCTL: track 0.00 -> 23.5 mm, vias 0 -> 2
- net Net-(R28-Pad1): track 22.4 -> 0.00 mm, vias 2 -> 0
- net /STEREO: track 0.00 -> 21.9 mm, vias 0 -> 3
- net Net-(Q3-C): track 2.20 -> 21.4 mm, vias 0 -> 2
- net /SA: track 0.00 -> 18.5 mm
- net Net-(U2A--): track 0.00 -> 17.8 mm, vias 0 -> 1
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Other:
- board text added: "38KHz PLL"
- board text added: "PD"
- board text added: "Quadrature Phase"
- board text added: "SA"
- board text added: "VCO_IN"
- board text added: "VCTL"
- board text removed: "38khz_PLL"
- board text removed: "Pilot_V"

Commit message: MPX V4基板作成
Parts:
- RV1, TP3, TP5: moved to F.Cu
- moved R81 10.3 mm to (79.0, 109.7), turned to 180 degrees
- moved R82 9.58 mm to (79.0, 111.4), turned to 0 degrees
- moved C50 8.30 mm to (79.7, 113.4), turned to 0 degrees
- moved RV1 2.02 mm to (83.8, 119.3)
- turned TP3 to 0 degrees
- turned TP5 to 0 degrees
Routing:
- net /38KHz-PLL: track 53.0 -> 59.7 mm, vias 2 -> 1
- net /38KHz-PLL-INV: track 46.1 -> 49.1 mm, vias 2 -> 1
- net Net-(D2-A): track 3.09 -> 3.10 mm, vias 0 -> 2
- net Net-(R1-Pad2): vias 0 -> 1
- added copper zone on In2.Cu, net +5V
- added copper zone on In1.Cu, net GND
- removed copper zone on In1.Cu, net +5V
- removed copper zone on In2.Cu, net GND
Other:
- board text added: "COMP"
- board text added: "SB"

Commit message: MPXV4基板発注
Other:
- board text added: "FM-MPX Decorder テストボード Ver.4.0 2026/10/10 Akira345"
- board text removed: "FM-MPX Decorder テストボード Ver.4.0 2026/10/XX Akira345"
Changed lines of the file:
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@@
 		)
 	)
-	(gr_text "FM-MPX Decorder テストボード Ver.4.0\n2026/10/XX Akira345"
+	(gr_text "FM-MPX Decorder テストボード Ver.4.0\n2026/10/10 Akira345"
 		(at 107.0864 98.298 90)
 		(layer "F.SilkS")
