File: FM-FRONTEND-JFET/FM-FRONTEND-JFET.kicad_sch (KiCad schematic)
At the start: 46 parts, among them J1 ANT-IN, J2 VC-01, J3 10.7MHz Filter, J4 IF_OUT, J5 GND, J6 VC-02, J7 +5V, J8 GND, J9 VC_GND, Q1 2SK3557, Q2 2SK3557, Q3 2SK3557, T1 Transformer_1P_1S

Commit message: IFTとPVCのフットプリントとシンボル作成。回路図反映。フロントエンドの回路をLTSpiceに合わせる
Parts:
- removed C14, C16, C17: 1000p, symbol Device:C_Small
- removed C15: 0.1u, symbol Device:C_Small
- removed D1: D_Capacitance, symbol Device:D_Capacitance
- removed FB4, FB5: FerriteBead_Small, symbol Device:FerriteBead_Small
- removed J2: VC-01, symbol Connector:Conn_01x03_Pin
- removed J6: VC-02, symbol Connector:Conn_01x03_Pin
- removed J9: VC_GND, symbol Connector:Conn_01x03_Pin
- removed L3: 220n, symbol Device:L_Small
- removed R6: 1M, symbol Device:R_Small
- removed RV1: 100k, symbol Device:R_Potentiometer
- removed T1: Transformer_1P_1S, symbol Device:Transformer_1P_1S
- added C18: 30p, MyLib:ALPS_FM_PVC, symbol MyLib:ALPS_PolyVaricon_2x30p
- added C20: 33p, Capacitor_SMD:C_0603_1608Metric_Pad1.08x0.95mm_HandSolder, symbol Device:C_Small
- added C21, C22: 1000p, Capacitor_SMD:C_0603_1608Metric_Pad1.08x0.95mm_HandSolder, symbol Device:C_Small
- added Q4: 2SK3557, Package_TO_SOT_SMD:SOT-23_Handsoldering, symbol Device:Q_NJFET_SDG
- added R7: 1Meg, Resistor_SMD:R_0603_1608Metric_Pad0.98x0.95mm_HandSolder, symbol Device:R_Small
- added R8: 470, Resistor_SMD:R_0603_1608Metric_Pad0.98x0.95mm_HandSolder, symbol Device:R_Small
- added R9: 100k, Resistor_SMD:R_0603_1608Metric_Pad0.98x0.95mm_HandSolder, symbol Device:R_Small
- added T1: IFT_7mmx7mm, MyLib:IFT_7mmx7mm, symbol MyLib:IFT_7mmx7mm
- C1, C10, C11, C12, C2, C3, C5, C6, C7, C8, C9: footprint (none) -> Capacitor_SMD:C_0603_1608Metric_Pad1.08x0.95mm_HandSolder
- C13: value 5p -> 1000p; footprint (none) -> Capacitor_SMD:C_0603_1608Metric_Pad1.08x0.95mm_HandSolder
- C4: value 5p -> 39p; footprint (none) -> MyLib:ALPS_FM_PVC
- FB1, FB2, FB3: footprint (none) -> Inductor_SMD:L_0603_1608Metric_Pad1.05x0.95mm_HandSolder
- J1, J3, J4, J5, J7, J8: footprint (none) -> Connector_PinHeader_2.54mm:PinHeader_1x03_P2.54mm_Vertical
- L1: value 220n -> 82n; footprint (none) -> Inductor_THT:L_Radial_L8.0mm_W8.0mm_P5.00mm_Neosid_SD8
- L2: value 220n -> 56n; footprint (none) -> Inductor_THT:L_Axial_L9.5mm_D4.0mm_P2.54mm_Vertical_Fastron_SMCC
- Q1, Q2, Q3: footprint (none) -> Package_TO_SOT_SMD:SOT-23_Handsoldering
- R1, R2, R3, R4, R5: footprint (none) -> Resistor_SMD:R_0603_1608Metric_Pad0.98x0.95mm_HandSolder
Connections:
- net GND: now also C18.5, C18.5, R7.2, R8.2, R9.2, T1.3 (SA)
- net at C11.1, L2.1, Q3.3 (G): now also C18.4
- net at C5.1, C6.1, FB1.2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: now also C4.1
- net at C11.2, C12.1, Q3.1 (S)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: now also C22.1; no longer C13.1
- net at L1.2, Q1.2 (D): now also C20.2, C21.1; no longer C4.1
- net at C4.2, Q2.3 (G), R3.1: now also C20.1
- net at J3.3 (Pin_3): now also T1.5 (SB)
- net at C3.1, C7.1, C8.1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: now also T1.1 (AA)
- net at C3.2, Q2.2 (D): now also T1.2 (AB)
- net at C10.1, C9.1, FB3.2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: now also Q4.2 (D)
- new net: C13.1, Q4.1 (S), R8.1
- new net: C22.2, Q4.3 (G), R9.1
- new net: C18.3, C21.2, R7.1
- no-connect marks 0 -> 1
Other:
- moved on the sheet: C1, C10, C11, C12, C2, C9, FB3, J1, L1, L2, Q1, Q3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

Commit message: フェライトビーズの型番を追記
Parts:
- FB1, FB2, FB3: value FerriteBead_Small -> MPZ1608S601ATA00
Other:
- note added: "受信周波数：76-95MHz バリコン：10p-30p L1: 0.6mmを内径5mmで4ターン長さ3.3mm L2: 0.6mmを内径5mmで3ターン長さ2.3mm T1 27T:9T"
Changed lines of the file:
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@@
 	(generator_version "10.0")
 	(paper "A4")
+	(text "受信周波数：76-95MHz\nバリコン：10p-30p\nL1: 0.6mmを内径5mmで4ターン長さ3.3mm\nL2: 0.6mmを内径5mmで3ターン長さ2.3mm\n\nT1\n27T:9T"
+		(exclude_from_sim no)
+		(at 35.56 87.884 0)
+		(effects
+			(font
+				(size 1.27 1.27)
+			)
+		)
+	)
 	(junction
 		(at 64.77 114.3)
@@
 			)
 		)
-		(property "Value" "FerriteBead_Small"
+		(property "Value" "MPZ1608S601ATA00"
 			(at 46.9519 22.86 90)
 			(show_name no)
@@
 			)
 		)
-		(property "Value" "FerriteBead_Small"
+		(property "Value" "MPZ1608S601ATA00"
 			(at 69.8119 91.44 90)
 			(show_name no)
@@
 			)
 		)
-		(property "Value" "FerriteBead_Small"
+		(property "Value" "MPZ1608S601ATA00"
 			(at 110.4519 22.86 90)
 			(show_name no)

Commit message: 回路ミス修正
Parts:
- added C14: 10p, Capacitor_SMD:C_0603_1608Metric_Pad1.08x0.95mm_HandSolder, symbol Device:C_Small
Connections:
- net GND: now also C14.2
- net at C11.1, C18.4, L2.1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: now also C14.1
Other:
- moved on the sheet: C18B, L2
