File: FM-IF-DET/FM-IF-DET.kicad_sch (KiCad schematic)
At the start: 101 parts, among them J1 IF-IN, J2 MPX-OUT, Q1 MMDT3904, Q10 MMBT3904, Q2 MMDT3904, Q3 MMDT3904, Q4 MMDT3904, Q5 MMBT3904, Q6 2SK3557, Q7 MMDT3904, Q8 MMDT3904, Q9 MMDT3904

Commit message: IFTとPVCのフットプリントとシンボル作成。回路図反映。フロントエンドの回路をLTSpiceに合わせる
Parts:
- removed L1: 2.21u, symbol Device:L_Small
- added T1: 2.21u, MyLib:IFT_7mmx7mm, symbol MyLib:IFT_7mmx7mm
- C1, C10, C11, C12, C13, C14, C15, C16, C17, C18, C19, C2, C20, C23, C24, C25, C26, C27, C28, C29, C3, C30, C31, C32, C4, C5, C6, C7, C8, C9: footprint (none) -> Capacitor_SMD:C_0603_1608Metric_Pad1.08x0.95mm_HandSolder
- C21, C22: footprint Resistor_THT:R_Array_SIP4 -> Capacitor_SMD:C_0603_1608Metric_Pad1.08x0.95mm_HandSolder
- R1, R10, R11, R12, R13, R14, R15, R16, R17, R18, R19, R2, R20, R21, R22, R23, R24, R25, R26, R27, R28, R29, R3, R30, R31, R32, R33, R34, R35, R4, R5, R50, R51, R52, R53, R54, R55, R56, R6, R7, R8, R9: footprint (none) -> Resistor_SMD:R_0603_1608Metric_Pad0.98x0.95mm_HandSolder
- R36, R37, R38, R39, R40, R41, R42, R43, R44, R45, R46, R47, R48, R49: footprint Package_TO_SOT_SMD:SOT-23 -> Resistor_SMD:R_0603_1608Metric_Pad0.98x0.95mm_HandSolder
Connections:
- net GND: now also T1.1 (AA)
- net at C23.2, C24.2, Q6.3 (G)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: now also T1.2 (AB)
- no-connect marks 0 -> 3

Commit message: 回路ミス修正
Connections:
- net OB: now also Q8.6 (C1); no longer Q8.3 (C2)
- net at C26.1, Q7.6 (C1), R45.2: now also Q8.3 (C2); no longer Q8.6 (C1)
Changed lines of the file:
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@@
+	)
+	(junction
+		(at 177.8 91.44)
+		(diameter 0)
+		(color 0 0 0 0)
 	)
 	(junction
@@
 	)
 	(junction
-		(at 177.8 93.98)
-		(diameter 0)
-		(color 0 0 0 0)
-	)
-	(junction
 		(at 64.77 34.29)
 		(diameter 0)
@@
 	)
 	(junction
-		(at 218.44 96.52)
+		(at 233.68 90.17)
 		(diameter 0)
 		(color 0 0 0 0)
@@
 	(junction
 		(at 233.68 91.44)
+		(diameter 0)
+		(color 0 0 0 0)
+	)
+	(junction
+		(at 209.55 90.17)
 		(diameter 0)
 		(color 0 0 0 0)
@@
 	(wire
 		(pts
-			(xy 177.8 93.98) (xy 209.55 93.98)
-		)
-		(stroke
-			(width 0)
-			(type default)
-		)
-	)
-	(wire
-		(pts
 			(xy 168.91 104.14) (xy 170.18 104.14)
 		)
@@
 	(wire
 		(pts
+			(xy 218.44 91.44) (xy 177.8 91.44)
+		)
+		(stroke
+			(width 0)
+			(type default)
+		)
+	)
+	(wire
+		(pts
 			(xy 157.48 55.88) (xy 157.48 58.42)
 		)
@@
 	(wire
 		(pts
+			(xy 233.68 90.17) (xy 233.68 91.44)
+		)
+		(stroke
+			(width 0)
+			(type default)
+		)
+	)
+	(wire
+		(pts
 			(xy 373.38 34.29) (xy 373.38 38.1)
 		)
@@
 	(wire
 		(pts
-			(xy 177.8 99.06) (xy 177.8 93.98)
-		)
-		(stroke
-			(width 0)
-			(type default)
-		)
-	)
-	(wire
-		(pts
-			(xy 218.44 96.52) (xy 218.44 99.06)
+			(xy 177.8 91.44) (xy 177.8 99.06)
 		)
 		(stroke
@@
 	(wire
 		(pts
+			(xy 186.69 90.17) (xy 209.55 90.17)
+		)
+		(stroke
+			(width 0)
+			(type default)
+		)
+	)
+	(wire
+		(pts
 			(xy 233.68 81.28) (xy 233.68 82.55)
 		)
@@
 	(wire
 		(pts
-			(xy 209.55 93.98) (xy 209.55 99.06)
-		)
-		(stroke
-			(width 0)
-			(type default)
-		)
-	)
-	(wire
-		(pts
 			(xy 138.43 50.8) (xy 140.97 50.8)
 		)
@@
 	(wire
 		(pts
+			(xy 218.44 99.06) (xy 218.44 91.44)
+		)
+		(stroke
+			(width 0)
+			(type default)
+		)
+	)
+	(wire
+		(pts
 			(xy 257.81 50.8) (xy 261.62 50.8)
 		)
@@
 	(wire
 		(pts
-			(xy 218.44 91.44) (xy 218.44 96.52)
-		)
-		(stroke
-			(width 0)
-			(type default)
-		)
-	)
-	(wire
-		(pts
 			(xy 128.27 50.8) (xy 128.27 55.88)
 		)
@@
 	(wire
 		(pts
-			(xy 177.8 91.44) (xy 177.8 93.98)
-		)
-		(stroke
-			(width 0)
-			(type default)
-		)
-	)
-	(wire
-		(pts
 			(xy 170.18 125.73) (xy 172.72 125.73)
 		)
@@
 	(wire
 		(pts
+			(xy 209.55 90.17) (xy 233.68 90.17)
+		)
+		(stroke
+			(width 0)
+			(type default)
+		)
+	)
+	(wire
+		(pts
 			(xy 106.68 138.43) (xy 106.68 139.7)
 		)
@@
 	(wire
 		(pts
-			(xy 186.69 96.52) (xy 218.44 96.52)
-		)
-		(stroke
-			(width 0)
-			(type default)
-		)
-	)
-	(wire
-		(pts
 			(xy 318.77 41.91) (xy 318.77 45.72)
 		)
@@
 	(wire
 		(pts
+			(xy 209.55 99.06) (xy 209.55 90.17)
+		)
+		(stroke
+			(width 0)
+			(type default)
+		)
+	)
+	(wire
+		(pts
 			(xy 162.56 97.79) (xy 162.56 101.6)
 		)
@@
 	(wire
 		(pts
-			(xy 186.69 99.06) (xy 186.69 96.52)
-		)
-		(stroke
-			(width 0)
-			(type default)
-		)
-	)
-	(wire
-		(pts
 			(xy 67.31 29.21) (xy 74.93 29.21)
 		)
@@
 	(wire
 		(pts
-			(xy 233.68 87.63) (xy 233.68 91.44)
+			(xy 233.68 87.63) (xy 233.68 90.17)
 		)
 		(stroke
@@
 	(wire
 		(pts
-			(xy 233.68 91.44) (xy 218.44 91.44)
-		)
-		(stroke
-			(width 0)
-			(type default)
-		)
-	)
-	(wire
-		(pts
 			(xy 312.42 34.29) (xy 314.96 34.29)
 		)
@@
 		)
 		(stroke
+			(width 0)
+			(type default)
+		)
+	)
+	(wire
+		(pts
+			(xy 186.69 99.06) (xy 186.69 90.17)
+		)
+		(stroke
