File: FM-Radio-Reciever/FM-Radio-Reciever.kicad_pcb (KiCad board)
At the start: 4 copper layers, 73 x 73 mm, 214 parts, among them J1 ANT-IN, J2 GND, J4 10.7MHz Filter, J5 GND, J6 MPX-OUT, J7 +5V, J8 GND, Q1 2SK3557, Q10 MMDT3904, Q11 MMDT3904, Q12 MMBT3904, Q13 MMDT3904, Q14 MMDT3904, Q15 MMDT3904, Q16 MMBT3904, Q2 2SK3557, Q3 2SK3557, Q4 2SK3557, Q5 2SK3557, Q6 MMBT3904, Q7 MMDT3904, Q8 MMDT3904, Q9 MMDT3904, SW1 AFC_SW, T1 2.21u, T2 IFT_7mm, U1 LM393

Commit message: フロントエンド、IF部分の基板設計
Parts:
- C14, C15, C25, C52: moved to B.Cu
- C43: moved to F.Cu
- moved D3 73.4 mm to (61.5, 171.8)
- moved C61 73.4 mm to (71.5, 152.8)
- moved C63 73.4 mm to (44.6, 159.4)
- moved D4 73.4 mm to (57.1, 171.8)
- moved R70 73.4 mm to (65.9, 116.2)
- moved R71 73.4 mm to (71.2, 163.2)
- moved R73 73.4 mm to (70.2, 158.0)
- moved R76 73.4 mm to (34.0, 173.3)
- moved R80 73.4 mm to (41.9, 173.6)
- moved R86 73.4 mm to (67.2, 162.1)
- moved R87 73.4 mm to (67.1, 158.5)
- moved R91 73.4 mm to (59.6, 169.4)
- moved RV1 73.4 mm to (67.7, 169.1)
- moved TP9 73.4 mm to (77.2, 169.1)
- moved C62 73.4 mm to (56.0, 158.0)
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Routing:
- net /VBias: track 0.00 -> 82.6 mm
- net Net-(Q5-G): track 0.00 -> 26.3 mm, vias 0 -> 1
- net Net-(Q3-G): track 0.00 -> 18.4 mm
- net Net-(Q3-S): track 0.00 -> 14.1 mm
- net Net-(Q3-D): track 0.00 -> 13.8 mm
- net Net-(JP2-A): track 0.00 -> 13.0 mm
- net Net-(Q1-D): track 0.00 -> 12.2 mm
- net Net-(Q4-S): track 0.00 -> 11.8 mm
- net /S4A: track 0.00 -> 11.6 mm
- net /S4B: track 0.00 -> 11.3 mm, vias 0 -> 2
- net Net-(J1-Pin_1): track 0.00 -> 9.93 mm
- net /S1B: track 0.00 -> 9.64 mm, vias 0 -> 2
- net /S2B: track 0.00 -> 9.59 mm, vias 0 -> 2
- net /S3B: track 0.00 -> 9.44 mm, vias 0 -> 2
- net Net-(C35-Pad1): track 0.00 -> 9.12 mm
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
Commit message: PCB設計いったん完了
Parts:
- C13, C23, C48, Q9, R15, R18, R19, R23, R61, R69: moved to B.Cu
- C17, C62, C63, C64, JP3, Q15, Q16, R10, R71, R72, R75, R76, R77, R78, R79, R80, R81, R82, R83, R87, R89, R9, R93, R94: moved to F.Cu
- T2: value IFT_7mm -> IFT_7mmx7mm
- moved R85 121.3 mm to (155.2, 162.9), turned to 180 degrees
- moved R94 112.7 mm to (150.6, 170.3), turned to 180 degrees
- moved R95 112.1 mm to (155.0, 169.9)
- moved R76 106.3 mm to (140.2, 168.8), turned to 90 degrees
- moved R78 104.7 mm to (138.7, 168.8), turned to -90 degrees
- moved R79 104.3 mm to (140.3, 160.4), turned to 90 degrees
- moved R93 104.3 mm to (148.0, 169.3), turned to 90 degrees
- moved R81 103.6 mm to (144.4, 163.1), turned to 0 degrees
- moved R80 102.9 mm to (144.4, 164.7)
- moved TP12 102.3 mm to (153.9, 159.3)
- moved JP3 101.6 mm to (138.6, 164.7)
- moved Q15 101.4 mm to (141.6, 164.8)
- moved D6 100.9 mm to (152.2, 170.8), turned to 0 degrees
- moved C62 100.8 mm to (148.6, 118.0), turned to -90 degrees
- moved R75 99.5 mm to (137.1, 160.4)
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Routing:
- net /DB: track 0.00 -> 91.5 mm, vias 0 -> 1
- net /DA: track 0.00 -> 82.9 mm, vias 0 -> 1
- net Net-(D2-K): track 0.00 -> 58.3 mm, vias 0 -> 1
- net Net-(D3-K): track 0.00 -> 47.1 mm, vias 0 -> 3
- net Net-(D4-K): track 0.00 -> 39.5 mm, vias 0 -> 2
- net /AFC_V: track 1.82 -> 40.6 mm
- net /S4A: track 11.6 -> 46.9 mm, vias 0 -> 3
- net /S4B: track 11.3 -> 45.9 mm
- net /OB: track 0.00 -> 19.5 mm, vias 0 -> 1
- net /VBL: track 0.00 -> 19.3 mm
- net /AFC_BIAS: track 0.00 -> 19.2 mm, vias 0 -> 1
- net /OA: track 0.00 -> 16.6 mm, vias 0 -> 2
- net /SF: track 0.00 -> 13.2 mm
- net /VBU: track 0.00 -> 12.8 mm
- net Net-(JP3-C): track 0.00 -> 11.9 mm
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Other:
- board text added: "TUNING PANEL (AFC/LED)"
- board text removed: "TUNING PANEL (AFC/LED drive on B side)"
