File: FM-Radio-Reciever/FM-Radio-Reciever.kicad_sch (KiCad schematic)
At the start: 214 parts, among them J1 ANT-IN, J2 GND, J3 RFShield_OnePiece, J4 10.7MHz Filter, J5 GND, J6 MPX-OUT, J7 +5V, J8 GND, Q1 2SK3557, Q10 MMDT3904, Q11 MMDT3904, Q12 MMBT3904, Q13 MMDT3904, Q14 MMDT3904, Q15 MMDT3904, Q16 MMBT3904, Q2 2SK3557, Q3 2SK3557, Q4 2SK3557, Q5 2SK3557, Q6 MMBT3904, Q7 MMDT3904, Q8 MMDT3904, Q9 MMDT3904, SW1 AFC_SW, T1 2.21u, T2 IFT_7mmx7mm, U1 LM393

Commit message: 部品配置をざっくり決める
Parts:
- removed J3: RFShield_OnePiece, RF_Shielding:Laird_Technologies_BMI-S-205-F_38.10x25.40mm, symbol Device:RFShield_OnePiece
- removed SW1: AFC_SW, Button_Switch_SMD:Nidec_Copal_CAS-120A, symbol Switch:SW_Nidec_CAS-120A1
- added JP3: AB-SWAP, Jumper:SolderJumper-3_P1.3mm_Bridged12_RoundedPad1.0x1.5mm, symbol Jumper:SolderJumper_3_Bridged12
- added SW1: AFC_SW, Button_Switch_THT:SW_Slide-03_Wuerth-WS-SLTV_10x2.5x6.4_P2.54mm, symbol Switch:SW_SPDT
- D1: footprint Diode_THT:D_A-405_P2.54mm_Vertical_AnodeUp -> Diode_THT:D_DO-35_SOD27_P2.54mm_Vertical_AnodeUp
- D5, D6: footprint Diode_SMD:D_0603_1608Metric_Pad1.05x0.95mm_HandSolder -> Diode_SMD:D_SOD-323_HandSoldering
- RV1: footprint Resistor_SMD:R_0603_1608Metric_Pad0.98x0.95mm_HandSolder -> Potentiometer_SMD:Potentiometer_Bourns_TC33X_Vertical
- TP1: value TestPoint -> OSC
- TP10: value TestPoint -> AFC_V
- TP11: value TestPoint -> DB
- TP12: value TestPoint -> DA
- TP2: value TestPoint -> IF
- TP3: value TestPoint -> SF
- TP4: value TestPoint -> LPF_OUT
- TP5: value TestPoint -> IF_OUT
- TP6: value TestPoint -> VBU
- TP7: value TestPoint -> VBL
- TP8: value TestPoint -> VBias
- TP9: value TestPoint -> AFC_BIAS
Connections:
- net AFC_BIAS: now also SW1.1 (A)
- net AFC_V: now also SW1.2 (B); no longer TP10.1
- net at Q15.3 (C2), R76.2, R78.1: now also JP3.1 (A); no longer C64.1
- net at Q15.6 (C1), R75.2, R77.2: now also JP3.3 (B)
- net at C9.2, R3.1: now also C8.4; no longer C8.3
- net at C10.1, C2.1, C59.1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: now also C8.3; no longer C8.4
- new net: C64.1, JP3.2 (C), SW1.3 (C), TP10.1
Other:
- moved on the sheet: C61, C62, C64, D2, D3, D4, D5, D6, J6, Q15A, Q15B, Q16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

Commit message: プロトタイプ基板発注
Connections:
- net Q_TANK: now reaches C13.2, C5.2, Q2.3 (G), R6.1, T1.2 (AB)
Other:
- note added: "位相シフト LT1は中華ボビン(Aitendo T7X7KA 内径 5mm) に0.21mmを17T その後コアを調整"
- note added: "受信周波数：76-95MHz バリコン：10p-30p L2: 0.6mmを内径5mmで4ターン長さ3.3mm L1: 0.6mmを内径5mmで3ターン長さ2.3mm T2 ボビン：Aitendo T7X7KA 巻き数比3:1 27T:9T (0.21mm)"
- note removed: "位相シフト LT1は中華ボビン(内径 5mm) に17T その後コアを調整"
- note removed: "受信周波数：76-95MHz バリコン：10p-30p L2: 0.6mmを内径5mmで4ターン長さ3.3mm L1: 0.6mmを内径5mmで3ターン長さ2.3mm T2 27T:9T"
Changed lines of the file:
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@@
 		)
 	)
-	(text "位相シフト\nLT1は中華ボビン(内径 5mm) に17T\nその後コアを調整"
+	(text "位相シフト\nLT1は中華ボビン(Aitendo T7X7KA 内径 5mm)\n に0.21mmを17T\nその後コアを調整"
 		(exclude_from_sim no)
-		(at 88.138 219.964 0)
+		(at 84.836 219.202 0)
 		(effects
 			(font
@@
 		)
 	)
-	(text "受信周波数：76-95MHz\nバリコン：10p-30p\nL2: 0.6mmを内径5mmで4ターン長さ3.3mm\nL1: 0.6mmを内径5mmで3ターン長さ2.3mm\n\nT2\n27T:9T"
+	(text "受信周波数：76-95MHz\nバリコン：10p-30p\nL2: 0.6mmを内径5mmで4ターン長さ3.3mm\nL1: 0.6mmを内径5mmで3ターン長さ2.3mm\n\nT2\nボビン：Aitendo T7X7KA 巻き数比3:1\n27T:9T (0.21mm)"
 		(exclude_from_sim no)
 		(at 35.814 78.74 0)
@@
 		(effects
 			(font
+				(size 1.27 1.27)
+			)
+			(justify left bottom)
+		)
+	)
+	(label "Q_TANK"
+		(at 81.28 231.14 0)
+		(effects
+			(font

Commit message: コンデンサの値間違い修正
Parts:
- C14: value 39p -> 33p
Changed lines of the file:
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@@
 		(dnp no)
 		(property "Reference" "C14"
-			(at 96.52 26.162 0)
+			(at 88.392 32.512 0)
 			(show_name no)
 			(do_not_autoplace no)
@@
 			)
 		)
-		(property "Value" "39p"
-			(at 96.52 27.94 0)
+		(property "Value" "33p"
+			(at 88.646 34.798 0)
 			(show_name no)
 			(do_not_autoplace no)
